Commit message: [fix] robot rotation

File: mio_robot/urdf/mio_robot.xacro (robot description, xacro)
@@ -123,5 +123,5 @@
     <parent link="base_link"/>
     <child link="caster_wheel"/>
-    <origin xyz="${caster_wheel_joint_offset} 0 -${caster_wheel_radius+0.005}" rpy="0 0 0"/>
+    <origin xyz="${caster_wheel_joint_offset} 0 -${caster_wheel_radius-0.005}" rpy="0 0 0"/>
   </joint>
   <xacro:property name="laser_size_x" value="0.03"/>
@@ -138,9 +138,4 @@
       <material name="blue"/>
     </visual>
-    <!--visual>
-      <geometry>
-        <mesh filename="package://mio_robot_description/meshes/hokuyo.dae"/>
-      </geometry>
-    </visual-->
     <collision>
       <geometry>
@@ -148,5 +143,5 @@
       </geometry>
     </collision>
-    <xacro:box_inertia m="0.2" w="${laser_size_x}" h="${laser_size_y}" d="${laser_size_z}"/>
+    <xacro:box_inertia m="12" w="${laser_size_x}" h="${laser_size_y}" d="${laser_size_z}"/>
   </link>
   <joint name="sensor_laser_joint" type="fixed">

File: mio_robot/urdf/mio_robot_gazebo_plugins.xacro (robot description, xacro)
@@ -9,7 +9,5 @@
             <leftJoint>left_wheel_joint</leftJoint>
             <rightJoint>right_wheel_joint</rightJoint>
-            <wheelSeparation>${wheel_separation}</wheelSeparation>
-            <wheelDiameter>${wheel_radius * 2}</wheelDiameter>
-            <torque>20</torque>
+            <wheelDiameter>0.08</wheelDiameter>
             <commandTopic>/cmd_vel</commandTopic>
             <odometryTopic>/odom</odometryTopic>

Commit message: [fix] xacro file

File: mio_robot/urdf/mio_robot.xacro (robot description, xacro)
@@ -123,5 +123,5 @@
     <parent link="base_link"/>
     <child link="caster_wheel"/>
-    <origin xyz="${caster_wheel_joint_offset} 0 -${caster_wheel_radius-0.005}" rpy="0 0 0"/>
+    <origin xyz="${caster_wheel_joint_offset} 0 -${caster_wheel_radius+0.005}" rpy="0 0 0"/>
   </joint>
   <xacro:property name="laser_size_x" value="0.03"/>
@@ -138,4 +138,9 @@
       <material name="blue"/>
     </visual>
+    <!--visual>
+      <geometry>
+        <mesh filename="package://mio_robot_description/meshes/hokuyo.dae"/>
+      </geometry>
+    </visual-->
     <collision>
       <geometry>
@@ -143,5 +148,5 @@
       </geometry>
     </collision>
-    <xacro:box_inertia m="12" w="${laser_size_x}" h="${laser_size_y}" d="${laser_size_z}"/>
+    <xacro:box_inertia m="0.2" w="${laser_size_x}" h="${laser_size_y}" d="${laser_size_z}"/>
   </link>
   <joint name="sensor_laser_joint" type="fixed">

File: mio_robot/urdf/mio_robot_gazebo_plugins.xacro (robot description, xacro)
@@ -9,5 +9,7 @@
             <leftJoint>left_wheel_joint</leftJoint>
             <rightJoint>right_wheel_joint</rightJoint>
-            <wheelDiameter>0.08</wheelDiameter>
+            <wheelSeparation>${wheel_separation}</wheelSeparation>
+            <wheelDiameter>${wheel_radius * 2}</wheelDiameter>
+            <torque>20</torque>
             <commandTopic>/cmd_vel</commandTopic>
             <odometryTopic>/odom</odometryTopic>

Commit message: minors

File: mio_robot/urdf/mio_robot.xacro (robot description, xacro)
@@ -56,4 +56,5 @@
     <xacro:box_inertia m="10" w="${base_len}" h="${base_width}" d="0.01"/>
     <visual>
+      <origin xyz="0 0 0.03" rpy="0 0 0" />
       <geometry>
         <box size="${base_len} ${base_width} 0.01"/>
@@ -77,5 +78,5 @@
     <link name="${prefix}_wheel">
       <visual>
-        <origin xyz="0 0 0" rpy="${pi/2} 0 0"/>
+        <origin xyz="0 0 0.032" rpy="${pi/2} 0 0"/>
         <geometry>
           <cylinder radius="${wheel_radius}" length="0.005"/>
@@ -155,4 +156,4 @@
     <child link="sensor_laser" />
   </joint>
-  <xacro:include filename="$(find mio_robot)/urdf/mio_robot_gazebo_plugins.xacro"/>
+<!--  <xacro:include filename="$(find mio_robot)/urdf/mio_robot_gazebo_plugins.xacro"/>-->
 </robot>

Commit message: minors

File: mio_robot/urdf/mio_robot.xacro (robot description, xacro)
@@ -56,5 +56,5 @@
     <xacro:box_inertia m="10" w="${base_len}" h="${base_width}" d="0.01"/>
     <visual>
-      <origin xyz="0 0 0.03" rpy="0 0 0" />
+      <origin xyz="0 0 0.03" rpy="-${pi} 0 ${pi}" />
       <geometry>
         <box size="${base_len} ${base_width} 0.01"/>
@@ -70,5 +70,5 @@
   <!--base_link to base_footprint Joint-->
   <joint name="base_link_joint" type="fixed">
-    <origin xyz="0 0 ${wheel_radius + 0.005}" rpy="0 0 0" />
+    <origin xyz="0 0 ${wheel_radius + 0.005}" rpy="-${pi} 0 ${pi}" />
     <parent link="base_footprint"/>
     <child link="base_link" />

File: mio_robot/urdf/mio_robot_gazebo_plugins.xacro (robot description, xacro)
@@ -21,5 +21,5 @@
         <material>Gazebo/FlatBlack</material>
         <sensor type="ray" name="lds_lfcd_sensor">
-            <pose>0 0 0 0 0 0</pose>
+            <pose>0 0 0 -${pi} 0 ${pi}</pose>
             <visualize>false</visualize>
             <update_rate>5</update_rate>
